Commit message: #update

File: robot_utils/urdf/arm.urdf (robot description, URDF)
Before this commit: robot gaze_arm, 5 links, 4 joints
Links:
- added link world
- link base_link: mass None -> 0.03; geometry collision cylinder length=0.088 radius=0.015; visual mesh filename=package://robot_utils/stl/base_link.STL
- link hand_link: mass None -> 0.03; geometry collision cylinder length=0.088 radius=0.015; visual box size=0.05 0.045 0.025
- link link1: mass None -> 0.03; geometry collision cylinder length=0.088 radius=0.015; visual mesh filename=package://robot_utils/stl/joint1.STL
- link link2: mass None -> 0.03; geometry collision cylinder length=0.088 radius=0.015; visual mesh filename=package://robot_utils/stl/link1.STL
- link link3: mass None -> 0.03; geometry collision cylinder length=0.088 radius=0.015; visual mesh filename=package://robot_utils/stl/link2.STL
Joints:
- added joint base_joint: type fixed, parent world, child base_link
- joint hand_joint: limit lower=-1.046666667 upper=1.046666667 effort=0.5293 velocity=6.159937255 -> lower=-1.57 upper=1.57 effort=0.5293 velocity=6.159937255
- joint joint2: limit lower=-1.046666667 upper=1.046666667 effort=0.5293 velocity=6.159937255 -> lower=-1.57 upper=1.57 effort=0.5293 velocity=6.159937255
